Commit message: fixes tf problem

File: p3dx_description/urdf/pioneer3dx.xacro (robot description, xacro)
@@ -18,190 +18,190 @@
  -->
 <robot name="pioneer3dx" xmlns:xacro="http://www.ros.org/xacro">
-  <!-- import the pioneer 3dx's wheels -->
-  <xacro:include filename="$(find p3dx_description)/urdf/pioneer3dx_wheel.xacro" />
-  <!-- import all gazebo-customization elements, including gazebo colors -->
-  <xacro:include filename="$(find p3dx_description)/urdf/pioneer3dx.gazebo" />
-  <!-- chassis -->
-    <link name="base_link">
-        <inertial>
-            <mass value="3.5" />
-            <origin xyz="-0.05 0 0" />
-            <inertia ixx="1" ixy="0" ixz="0" iyy="1" iyz="0" izz="1" />
-        </inertial>
-        <visual>
-            <origin xyz="-0.045 0 0.148" rpy="0 0 0" />
-            <geometry name="pioneer_geom">
-                <mesh filename="package://p3dx_description/meshes/chassis.stl" />
-            </geometry>
-        </visual>
-        <collision>
-            <origin xyz="-0.045 0 0.145" rpy="0 0 0" />
-            <geometry>
-                <box size="0.35 0.25 0.14" />
-            </geometry>
-        </collision>
-    </link>
-  <!-- top_plate -->
-    <link name="top_plate">
-        <inertial>
-            <mass value="0.01" />
-            <origin xyz="0 0 0" />
-            <inertia ixx="1" ixy="0" ixz="0" iyy="1" iyz="0" izz="1" />
-        </inertial>
-        <visual>
-            <origin xyz="0 0 0" rpy="0 0 0" />
-            <geometry name="top_geom">
-                <mesh filename="package://p3dx_description/meshes/top.stl" />
-            </geometry>
-        </visual>
-        <collision>
-            <origin xyz="0.0 0 0" rpy="0 0 0" />
-            <geometry name="pioneer_geom">
-                <box size="0.45 0.38 0.01" />
-            </geometry>
-        </collision>
-    </link>
-    <joint name="base_top_joint" type="fixed">
-        <origin xyz="-0.045 0 0.234" rpy="0 0 0" />
-        <parent link="base_link" />
-        <child link="top_plate" />
-    </joint>
-  <!-- swivel -->
-    <link name="swivel">
-        <inertial>
-            <mass value="0.1" />
-            <origin xyz="0 0 0" />
-            <inertia ixx="0.01" ixy="0" ixz="0" iyy="0.01" iyz="0" izz="0.01" />
-        </inertial>
-        <visual>
-            <origin xyz="0 0 0" rpy="0 0 0" />
-            <geometry name="pioneer_geom">
-                <mesh filename="package://p3dx_description/meshes/swivel.stl" />
-            </geometry>
-        </visual>
-        <collision>
-            <origin xyz="0 0 0" rpy="0 0 0" />
-            <geometry>
-                <box size="0 0 0" />
-            </geometry>
-        </collision>
-    </link>
-    <joint name="base_swivel_joint" type="continuous">
-        <origin xyz="-0.185 0 0.055" rpy="0 0 0" />
-        <axis xyz="0 0 1" />
-        <anchor xyz="0 0 0" />
-        <limit effort="100" velocity="100" k_velocity="0" />
-        <joint_properties damping="0.0" friction="0.0" />
-        <parent link="base_link" />
-        <child link="swivel" />
-    </joint>
-  <!-- center_hubcap -->
-    <link name="center_hubcap">
-        <inertial>
-            <mass value="0.01" />
-            <origin xyz="0 0 0" />
-            <inertia ixx="0.012411765597" ixy="-0.000711733678" ixz="0.00050272983"
-                iyy="0.015218160428" iyz="-0.000004273467" izz="0.011763977943" />
-        </inertial>
-        <visual>
-            <origin xyz="0 0 0" rpy="0 0 0" />
-            <geometry name="pioneer_geom">
-                <mesh filename="package://p3dx_description/meshes/center_hubcap.stl" />
-            </geometry>
-        </visual>
-        <collision>
-            <origin xyz="0 0 0" rpy="0 0 0" />
-            <geometry>
-                <box size="0 0 0" />
-            </geometry>
-        </collision>
-    </link>
-    <joint name="swivel_hubcap_joint" type="continuous">
-        <origin xyz="-0.026 0 -0.016" rpy="0 0 0" />
-        <axis xyz="0 1 0" />
-        <anchor xyz="0 0 0" />
-        <limit effort="100" velocity="100" k_velocity="0" />
-        <joint_properties damping="0.0" friction="0.0" />
-        <parent link="swivel" />
-        <child link="center_wheel" />
-    </joint>
-  <!-- center_wheel -->
-    <link name="center_wheel">
-        <inertial>
-            <mass value="0.1" />
-            <origin xyz="0 0 0" />
-            <inertia ixx="0.012411765597" ixy="-0.000711733678" ixz="0.00050272983"
-                iyy="0.015218160428" iyz="-0.000004273467" izz="0.011763977943" />
-        </inertial>
-        <visual>
-            <origin xyz="0 0 0" rpy="0 0 0" />
-            <geometry name="pioneer_geom">
-                <mesh filename="package://p3dx_description/meshes/center_wheel.stl" />
-            </geometry>
-        </visual>
-        <collision>
-            <origin xyz="0 0 0" rpy="${-3.1415927/2.0} 0 0" />
-            <geometry>
-                <cylinder radius="0.0375" length="0.01" />
-            </geometry>
-        </collision>
-    </link>
-    <joint name="center_wheel_joint" type="fixed">
-        <origin xyz="-0.0035 0 -0.001" rpy="0 0 0"/>
-        <parent link="center_wheel"/>
-        <child link="center_hubcap"/>
-    </joint>
-    <xacro:p3dx_wheel suffix="left" parent="base_link" reflect="1"/>
-    <xacro:p3dx_wheel suffix="right" parent="base_link" reflect="-1"/>
-  <!-- front_sonar -->
-    <link name="front_sonar">
-        <inertial>
-            <mass value="0.0001" />
-            <origin xyz="0 0 0" />
-            <inertia ixx="1" ixy="0" ixz="0" iyy="1" iyz="0" izz="1" />
-        </inertial>
-        <visual>
-            <origin rpy="0 0 0" xyz="0 0 0" />
-            <geometry name="pioneer_geom">
-                <mesh filename="package://p3dx_description/meshes/front_sonar.stl" />
-            </geometry>
-        </visual>
-        <collision>
-            <origin rpy="0 0 0" xyz="0 0 0" />
-            <geometry>
-                <box size="0 0 0" />
-            </geometry>
-        </collision>
-    </link>
-    <joint name="base_front_joint" type="fixed">
-        <origin rpy="0 0 0" xyz="0.109 0 0.209" />
-        <parent link="base_link" />
-        <child link="front_sonar" />
-    </joint>
-    <!-- lms100 laser -->
-    <link name="lms100">
-        <inertial>
-            <mass value="1e-5" />
-            <origin xyz="0 0 0" rpy="0 0 0" />
-            <inertia ixx="1e-6" ixy="0" ixz="0" iyy="1e-6" iyz="0" izz="1e-6" />
-        </inertial>
-        <visual>
-            <origin xyz="0 0 0" rpy="0 0 0" />
-            <geometry>
-                <mesh filename="package://p3dx_description/meshes/lms100.dae" />
-            </geometry>
-        </visual>
-        <collision>
-            <origin xyz="0 0 0" rpy="0 0 0" />
-            <geometry>
-                <box size="0.1 0.1 0.1" />
-            </geometry>
-        </collision>
-    </link>
-    <joint name="lms100_joint" type="fixed">
-        <axis xyz="0 1 0" />
-        <origin xyz="0.16 0 0.15" rpy="0 0 0" />
-        <parent link="base_link" />
-        <child link="lms100" />
-    </joint>
+<!-- import the pioneer 3dx's wheels -->
+<xacro:include filename="$(find p3dx_description)/urdf/pioneer3dx_wheel.xacro" />
+<!-- import all gazebo-customization elements, including gazebo colors -->
+<xacro:include filename="$(find p3dx_description)/urdf/pioneer3dx.gazebo" />
+<!-- chassis -->
+<link name="base_link">
+    <visual>
+        <origin xyz="-0.045 0 0.148" rpy="0 0 0" />
+        <geometry name="pioneer_geom">
+            <mesh filename="package://p3dx_description/meshes/chassis.stl" />
+        </geometry>
+    </visual>
+    <collision>
+        <origin xyz="-0.045 0 0.145" rpy="0 0 0" />
+        <geometry>
+            <box size="0.35 0.25 0.14" />
+        </geometry>
+    </collision>
+    <inertial>
+        <mass value="3.5" />
+        <origin xyz="-0.05 0 0" />
+        <inertia ixx="1" ixy="0" ixz="0" iyy="1" iyz="0" izz="1" />
+    </inertial>
+</link>
+<!-- top_plate -->
+<link name="top_plate">
+    <visual>
+        <origin xyz="0 0 0" rpy="0 0 0" />
+        <geometry name="top_geom">
+            <mesh filename="package://p3dx_description/meshes/top.stl" />
+        </geometry>
+    </visual>
+    <collision>
+        <origin xyz="0.0 0 0" rpy="0 0 0" />
+        <geometry name="pioneer_geom">
+            <box size="0.45 0.38 0.01" />
+        </geometry>
+    </collision>
+    <inertial>
+        <mass value="0.01" />
+        <origin xyz="0 0 0" />
+        <inertia ixx="1" ixy="0" ixz="0" iyy="1" iyz="0" izz="1" />
+    </inertial>
+</link>
+<joint name="base_top_joint" type="fixed">
+    <origin xyz="-0.045 0 0.234" rpy="0 0 0" />
+    <parent link="base_link" />
+    <child link="top_plate" />
+</joint>
+<!-- swivel -->
+<link name="swivel">
+    <visual>
+        <origin xyz="0 0 0" rpy="0 0 0" />
+        <geometry name="pioneer_geom">
+            <mesh filename="package://p3dx_description/meshes/swivel.stl" />
+        </geometry>
+    </visual>
+    <collision>
+        <origin xyz="0 0 0" rpy="0 0 0" />
+        <geometry>
+            <box size="0 0 0" />
+        </geometry>
+    </collision>
+    <inertial>
+        <mass value="0.1" />
+        <origin xyz="0 0 0" />
+        <inertia ixx="0.01" ixy="0" ixz="0" iyy="0.01" iyz="0" izz="0.01" />
+    </inertial>
+</link>
+<joint name="base_swivel_joint" type="fixed">
+    <origin xyz="-0.185 0 0.055" rpy="0 0 0" />
+    <axis xyz="0 0 1" />
+    <anchor xyz="0 0 0" />
+    <limit effort="100" velocity="100" k_velocity="0" />
+    <joint_properties damping="0.0" friction="0.0" />
+    <parent link="base_link" />
+    <child link="swivel" />
+</joint>
+<!-- center_hubcap -->
+<link name="center_hubcap">
+    <visual>
+        <origin xyz="0 0 0" rpy="0 0 0" />
+        <geometry name="pioneer_geom">
+            <mesh filename="package://p3dx_description/meshes/center_hubcap.stl" />
+        </geometry>
+    </visual>
+    <collision>
+        <origin xyz="0 0 0" rpy="0 0 0" />
+        <geometry>
+            <box size="0 0 0" />
+        </geometry>
+    </collision>
+    <inertial>
+        <mass value="0.01" />
+        <origin xyz="0 0 0" />
+        <inertia ixx="0.012411765597" ixy="-0.000711733678" ixz="0.00050272983"
+            iyy="0.015218160428" iyz="-0.000004273467" izz="0.011763977943" />
+    </inertial>
+</link>
+<joint name="swivel_hubcap_joint" type="fixed">
+    <origin xyz="-0.026 0 -0.016" rpy="0 0 0" />
+    <axis xyz="0 1 0" />
+    <anchor xyz="0 0 0" />
+    <limit effort="100" velocity="100" k_velocity="0" />
+    <joint_properties damping="0.0" friction="0.0" />
+    <parent link="swivel" />
+    <child link="center_wheel" />
+</joint>
+<!-- center_wheel -->
+<link name="center_wheel">
+    <visual>
+        <origin xyz="0 0 0" rpy="0 0 0" />
+        <geometry name="pioneer_geom">
+            <mesh filename="package://p3dx_description/meshes/center_wheel.stl" />
+        </geometry>
+    </visual>
+    <collision>
+        <origin xyz="0 0 0" rpy="${-3.1415927/2.0} 0 0" />
+        <geometry>
+            <cylinder radius="0.0375" length="0.01" />
+        </geometry>
+    </collision>
+    <inertial>
+        <mass value="0.1" />
+        <origin xyz="0 0 0" />
+        <inertia ixx="0.012411765597" ixy="-0.000711733678" ixz="0.00050272983"
+            iyy="0.015218160428" iyz="-0.000004273467" izz="0.011763977943" />
+    </inertial>
+</link>
+<joint name="center_wheel_joint" type="fixed">
+    <origin xyz="-0.0035 0 -0.001" rpy="0 0 0"/>
+    <parent link="center_wheel"/>
+    <child link="center_hubcap"/>
+</joint>
+<xacro:p3dx_wheel suffix="left" parent="base_link" reflect="1"/>
+<xacro:p3dx_wheel suffix="right" parent="base_link" reflect="-1"/>
+<!-- front_sonar -->
+<link name="front_sonar">
+    <visual>
+        <origin rpy="0 0 0" xyz="0 0 0" />
+        <geometry name="pioneer_geom">
+            <mesh filename="package://p3dx_description/meshes/front_sonar.stl" />
+        </geometry>
+    </visual>
+    <collision>
+        <origin rpy="0 0 0" xyz="0 0 0" />
+        <geometry>
+            <box size="0 0 0" />
+        </geometry>
+    </collision>
+    <inertial>
+        <mass value="0.0001" />
+        <origin xyz="0 0 0" />
+        <inertia ixx="1" ixy="0" ixz="0" iyy="1" iyz="0" izz="1" />
+    </inertial>
+</link>
+<joint name="base_front_joint" type="fixed">
+    <origin rpy="0 0 0" xyz="0.109 0 0.209" />
+    <parent link="base_link" />
+    <child link="front_sonar" />
+</joint>
+<!-- lms100 laser -->
+<link name="lms100">
+    <inertial>
+        <mass value="1e-5" />
+        <origin xyz="0 0 0" rpy="0 0 0" />
+        <inertia ixx="1e-6" ixy="0" ixz="0" iyy="1e-6" iyz="0" izz="1e-6" />
+    </inertial>
+    <visual>
+        <origin xyz="0 0 0" rpy="0 0 0" />
+        <geometry>
+            <mesh filename="package://p3dx_description/meshes/lms100.dae" />
+        </geometry>
+    </visual>
+    <collision>
+        <origin xyz="0 0 0" rpy="0 0 0" />
+        <geometry>
+            <box size="0.1 0.1 0.1" />
+        </geometry>
+    </collision>
+</link>
+<joint name="lms100_joint" type="fixed">
+    <axis xyz="0 1 0" />
+    <origin xyz="0.16 0 0.15" rpy="0 0 0" />
+    <parent link="base_link" />
+    <child link="lms100" />
+</joint>
 </robot>

Commit message: add rviz colors to pioneer robot

File: p3dx_description/urdf/pioneer3dx.xacro (robot description, xacro)
@@ -22,4 +22,6 @@
 <!-- import all gazebo-customization elements, including gazebo colors -->
 <xacro:include filename="$(find p3dx_description)/urdf/pioneer3dx.gazebo" />
+<!-- import materials to add color to the pioneer in rviz -->
+<xacro:include filename="$(find p3dx_description)/urdf/materials.xacro" />
 <!-- chassis -->
 <link name="base_link">
@@ -29,4 +31,5 @@
             <mesh filename="package://p3dx_description/meshes/chassis.stl" />
         </geometry>
+        <material name="ChassisRed"/>
     </visual>
     <collision>
@@ -49,4 +52,5 @@
             <mesh filename="package://p3dx_description/meshes/top.stl" />
         </geometry>
+        <material name="TopBlack"/>
     </visual>
     <collision>
@@ -74,4 +78,5 @@
             <mesh filename="package://p3dx_description/meshes/swivel.stl" />
         </geometry>
+        <material name="SwivelGrey"/>
     </visual>
     <collision>
@@ -103,4 +108,5 @@
             <mesh filename="package://p3dx_description/meshes/center_hubcap.stl" />
         </geometry>
+        <material name="HubcapYellow"/>
     </visual>
     <collision>
@@ -133,4 +139,5 @@
             <mesh filename="package://p3dx_description/meshes/center_wheel.stl" />
         </geometry>
+        <material name="WheelBlack"/>
     </visual>
     <collision>
@@ -161,4 +168,5 @@
             <mesh filename="package://p3dx_description/meshes/front_sonar.stl" />
         </geometry>
+        <material name="SonarYellow"/>
     </visual>
     <collision>

File: p3dx_description/urdf/pioneer3dx_wheel.xacro (robot description, xacro)
@@ -27,4 +27,5 @@
                 <mesh filename="package://p3dx_description/meshes/${suffix}_wheel.stl" />
             </geometry>
+            <material name="WheelBlack"/>
         </visual>
         <collision>
@@ -59,4 +60,5 @@
                 <mesh filename="package://p3dx_description/meshes/${suffix}_hubcap.stl" />
             </geometry>
+            <material name="HubcapYellow"/>
         </visual>
         <collision>

Commit message: set swivel_hubcap_joint and base_swivel_joint joints as continuous, lower update_rate for laser scanner

File: p3dx_description/urdf/pioneer3dx.xacro (robot description, xacro)
@@ -92,5 +92,5 @@
     </inertial>
 </link>
-<joint name="base_swivel_joint" type="fixed">
+<joint name="base_swivel_joint" type="continuous">
     <origin xyz="-0.185 0 0.055" rpy="0 0 0" />
     <axis xyz="0 0 1" />
@@ -123,5 +123,5 @@
     </inertial>
 </link>
-<joint name="swivel_hubcap_joint" type="fixed">
+<joint name="swivel_hubcap_joint" type="continuous">
     <origin xyz="-0.026 0 -0.016" rpy="0 0 0" />
     <axis xyz="0 1 0" />
